Commit message: Add reconfigurable gaits to urdf

File: panthera_description/urdf/panthera.urdf (robot description, URDF)
Before this commit: robot panthera, 13 links, 12 joints
Links:
- added link base_footprint
- link base_link: mass None -> 1; geometry collision box size=0.20597 0.216606 0.169247; visual box size=0.20597 0.216606 0.169247
Joints:
- added joint base_joint: type fixed, parent base_footprint, child base_link, origin xyz=0.0 0.0 0.010 rpy=0 0 0
- joint base_left_joint: axis (none) -> 0 1 0; limit (none) -> lower=0 upper=0.2 effort=10.0 velocity=0.1; type fixed -> prismatic
- joint base_right_joint: axis (none) -> 0 1 0; limit (none) -> lower=-0.2 upper=0 effort=10.0 velocity=0.1; type fixed -> prismatic
